File: garnet_hardware/garnet.kicad_sch (KiCad schematic)
At the start: 9 parts, among them J2 Conn_01x03_Pin, J3 actuator PTC, J4 batt PTC, J9 Micro_SD_Card, U1 ESP32-S3-MINI-1U

Commit message: added part numbers for H-bridge, started on PCB layout
Parts:
- R3, R4, R5: footprint (none) -> Resistor_SMD:R_0603_1608Metric_Pad0.98x0.95mm_HandSolder
- TP1: footprint (none) -> Connector_PinHeader_2.54mm:PinHeader_1x01_P2.54mm_Vertical
Other:
- sheet pezio sense ports: added CNVST1, SCLK1, SDI1, SDO1; removed none
Changed lines of the file:
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@@
 			)
 		)
-		(property "Footprint" ""
+		(property "Footprint" "Resistor_SMD:R_0603_1608Metric_Pad0.98x0.95mm_HandSolder"
 			(at 50.292 130.81 90)
 			(hide yes)
@@
 			)
 		)
-		(property "Footprint" ""
+		(property "Footprint" "Resistor_SMD:R_0603_1608Metric_Pad0.98x0.95mm_HandSolder"
 			(at 50.292 160.02 90)
 			(hide yes)
@@
 			)
 		)
-		(property "Footprint" ""
+		(property "Footprint" "Resistor_SMD:R_0603_1608Metric_Pad0.98x0.95mm_HandSolder"
 			(at 104.902 67.31 90)
 			(hide yes)
@@
 			)
 		)
-		(property "Footprint" ""
+		(property "Footprint" "Connector_PinHeader_2.54mm:PinHeader_1x01_P2.54mm_Vertical"
 			(at 104.14 68.58 0)
 			(hide yes)
@@
 	(sheet
 		(at 77.47 147.32)
-		(size 21.59 11.43)
+		(size 21.59 30.48)
 		(exclude_from_sim no)
 		(in_bom yes)
@@
 		)
 		(property "Sheetfile" "pezio sence.kicad_sch"
-			(at 77.47 159.3346 0)
+			(at 77.47 178.3846 0)
 			(show_name no)
 			(do_not_autoplace no)
@@
 			)
 		)
+		(pin "CNVST1" output
+			(at 99.06 149.86 0)
+			(effects
+				(font
+					(size 1.27 1.27)
+				)
+				(justify right)
+			)
+		)
+		(pin "SCLK1" input
+			(at 99.06 152.4 0)
+			(effects
+				(font
+					(size 1.27 1.27)
+				)
+				(justify right)
+			)
+		)
+		(pin "SDI1" input
+			(at 99.06 154.94 0)
+			(effects
+				(font
+					(size 1.27 1.27)
+				)
+				(justify right)
+			)
+		)
+		(pin "SDO1" output
+			(at 99.06 157.48 0)
+			(effects
+				(font
+					(size 1.27 1.27)
+				)
+				(justify right)
+			)
+		)

Commit message: power frount end and sd card layed out on PCB
Parts:
- added C39, C40: 1uF, Capacitor_SMD:C_0603_1608Metric_Pad1.08x0.95mm_HandSolder, symbol Device:C
- added J13: SD_A, Connector_Card:microSD_HC_Molex_47219-2001, symbol Connector:Micro_SD_Card
- added R41, R41-45, R41-46, R42, R43, R44, R45, R46, R47, R48: 10K, Resistor_SMD:R_0603_1608Metric_Pad0.98x0.95mm_HandSolder, symbol Device:R
- J2: value Conn_01x03_Pin -> USB; footprint (none) -> Connector_PinHeader_2.54mm:PinHeader_1x03_P2.54mm_Vertical
- J3, J4: footprint (none) -> Connector_PinHeader_2.54mm:PinHeader_1x02_P2.54mm_Horizontal
- J9: value Micro_SD_Card -> SD_A; footprint (none) -> Connector_Card:microSD_HC_Molex_47219-2001
Connections:
- net +3V3: now also J9.4 (VDD), C39.1, C40.1, J13.4 (VDD), R41-45.1, R41-46.1, R41.1, R42.1, R43.1, R44.1, R45.1, R46.1, R47.1, R48.1
- net GND: now also J9.6 (VSS), J9.SH (SHIELD), C39.2, C40.2, J13.6 (VSS), J13.SH (SHIELD)
- net actuator PTC: now also U1.18 (IO14); no longer U1.5 (IO1)
- net batt PTC: now also U1.7 (IO3); no longer U1.4 (IO0)
- net DAT2_A: now reaches J9.1 (DAT2)
- net DAT2_A: now also U1.10 (IO6), R41-45.2
- net DAT3_A: now reaches J9.2 (DAT3/CD)
- net DAT3_A: now also U1.11 (IO7), R44.2
- net CMD_A: now reaches J9.3 (CMD)
- net CMD_A: now also U1.6 (IO2), R43.2
- net CLK_A: now reaches J9.5 (CLK)
- net CLK_A: now also U1.30 (IO48)
- net DAT0_A: now reaches J9.7 (DAT0)
- net DAT0_A: now also U1.8 (IO4), R42.2
- net DAT1_A: now reaches J9.8 (DAT1)
- net DAT1_A: now also U1.9 (IO5), R41.2
- net CLK_B: now reaches U1.12 (IO8)
- net CLK_B: now also J13.5 (CLK)
- net CMD_B: now reaches U1.13 (IO9)
- net CMD_B: now also J13.3 (CMD), R47.2
- net DAT0_B: now reaches U1.14 (IO10)
- net DAT0_B: now also J13.7 (DAT0), R46.2
- net DAT1_B: now reaches U1.15 (IO11)
- net DAT1_B: now also J13.8 (DAT1), R45.2
- net DAT2_B: now reaches U1.16 (IO12)
- net DAT2_B: now also J13.1 (DAT2), R41-46.2
- net DAT3_B: now reaches U1.17 (IO13)
- net DAT3_B: now also J13.2 (DAT3/CD), R48.2
- net CNVST1: now reaches U1.19 (IO15)
- net SCLK1: now reaches U1.20 (IO16)
- net SDI1: now reaches U1.21 (IO17)
- net SCLK0: now reaches U1.22 (IO18)
- net SDI0: now reaches U1.25 (IO21)
- net actuator drive/LINB: now reaches U1.27 (IO47)
- net SDO1: now reaches U1.28 (IO33)
- net SDO0: now reaches U1.29 (IO34)
- net CNVST0: now reaches U1.31 (IO35)
- net actuator drive/HINA: now reaches U1.38 (IO42)
- net actuator drive/HINB: now reaches U1.41 (IO45)
- net actuator drive/LINA: now reaches U1.44 (IO46)
- new net Vsense: U1.5 (IO1)
Other:
- sheet actuator drive ports: added HINA, HINB, LINA, LINB; removed none
- sheet pezio sense ports: added CNVST0, SCLK0, SDI0, SDO0; removed none
- moved on the sheet: J9

Commit message: cleaned SPI lines, replaced MOSFETS with more sutible ones, added free wheeling diodes added current sensing
Parts:
- removed C40: 1uF, Capacitor_SMD:C_0603_1608Metric_Pad1.08x0.95mm_HandSolder, symbol Device:C
- removed J13: SD_A, Connector_Card:microSD_HC_Molex_47219-2001, symbol Connector:Micro_SD_Card
- removed R41-46, R45, R46, R47, R48: 10K, Resistor_SMD:R_0603_1608Metric_Pad0.98x0.95mm_HandSolder, symbol Device:R
- added C25, C27, C28, C29, C31, C32: TBD, Capacitor_SMD:C_0603_1608Metric_Pad1.08x0.95mm_HandSolder, symbol Device:C
- added R28, R29, R31, R33, R34, R35: 33R, Resistor_SMD:R_0603_1608Metric_Pad0.98x0.95mm_HandSolder, symbol Device:R
Connections:
- net CNVST0: now also R33.2
- net CNVST1: now also R28.2
- net GND: now also C25.2, C27.2, C28.2, C29.2, C31.2, C32.2
- net SCLK0: now also R34.2
- net SCLK1: now also R29.2
- net SDI0: now also R35.2
- net SDI1: now also R31.2
- net CLK_B: no longer names the net of U1.12 (IO8)
- net CMD_B: no longer names the net of U1.13 (IO9)
- net DAT0_B: no longer names the net of U1.14 (IO10)
- net DAT1_B: no longer names the net of U1.15 (IO11)
- net DAT2_B: no longer names the net of U1.16 (IO12)
- net DAT3_B: no longer names the net of U1.17 (IO13)
- new net pezio sense/CNVST0: C32.1, R33.1
- new net pezio sense/CNVST1: C28.1, R28.1
- new net pezio sense/SCLK0: C31.1, R34.1
- new net pezio sense/SCLK1: C27.1, R29.1
- new net pezio sense/SDI0: C29.1, R35.1
- new net pezio sense/SDI1: C25.1, R31.1
